Commit message: first humble commit

File: description/lidar.xacro (robot description, xacro)
@@ -4,5 +4,5 @@
         <parent link="chassis"/>
         <child link="laser_frame"/>
-        <origin xyz="0.122 0 0.212" rpy="0 0 0"/>
+        <origin xyz="0.122 0 0.212" rpy="0 0 3.14"/>
     </joint>
     <link name="laser_frame">

File: description/ros2_control.xacro (robot description, xacro)
@@ -4,5 +4,5 @@
         <ros2_control name="RealRobot" type="system">
             <hardware>
-                <plugin>diffdrive_arduino/DiffDriveArduinoHardware</plugin>
+                <plugin>diffdrive_arduino/DiffDriveArduino</plugin>
                 <param name="left_wheel_name">left_wheel_joint</param>
                 <param name="right_wheel_name">right_wheel_joint</param>

Commit message: re-rotated lidar

File: description/lidar.xacro (robot description, xacro)
@@ -4,5 +4,5 @@
         <parent link="chassis"/>
         <child link="laser_frame"/>
-        <origin xyz="0.122 0 0.212" rpy="0 0 3.14"/>
+        <origin xyz="0.122 0 0.212" rpy="0 0 0"/>
     </joint>
     <link name="laser_frame">

Commit message: rotated robot 180 degrees

File: description/lidar.xacro (robot description, xacro)
@@ -26,5 +26,5 @@
         </collision>
         <xacro:inertial_cylinder mass="0.1" length="0.04" radius="0.05">
-            <origin xyz="0 0 0" rpy="0 0 0"/>
+            <origin xyz="0 0 0" rpy="0 0 3.1415"/>
         </xacro:inertial_cylinder>
     </link>

File: description/robot_core.xacro (robot description, xacro)
@@ -38,5 +38,5 @@
         <parent link="base_link"/>
         <child link="base_footprint"/>
-        <origin xyz="0 0 0" rpy="0 0 0"/>
+        <origin xyz="0 0 0" rpy="0 0 3.1415"/>
     </joint>
     <link name="base_footprint">

File: description/ros2_control.xacro (robot description, xacro)
@@ -59,4 +59,21 @@
             <parameters>$(find clearo)/config/gaz_ros2_ctl_use_sim.yaml</parameters>
         </plugin>
+        <!-- <plugin filename="libgz-sim-diff-drive-system.so" name="gz::sim::systems::DiffDrive">
+            <right_joint>right_wheel_joint</right_joint>
+            <left_joint>left_wheel_joint</left_joint>
+            <wheel_separation>0.32</wheel_separation>
+            <wheel_radius>0.04</wheel_radius>
+            <max_linear_acceleration>10</max_linear_acceleration>
+            <odom_publish_frequency>100</odom_publish_frequency>
+            <topic>cmd_vel</topic>
+            <odom_topic>odom</odom_topic>
+            <frame_id>odom</frame_id>
+            <child_frame_id>base_link</child_frame_id>
+        </plugin>
+        <plugin filename="gz-sim-joint-state-publisher-system" name="gz::sim::systems::JointStatePublisher">
+            <topic>joint_states</topic>
+            <joint_name>right_wheel_joint</joint_name>
+            <joint_name>left_wheel_joint</joint_name>
+        </plugin> -->
     </gazebo>
 </robot>

Commit message: 180 degree re-orientation

File: description/lidar.xacro (robot description, xacro)
@@ -4,5 +4,5 @@
         <parent link="chassis"/>
         <child link="laser_frame"/>
-        <origin xyz="0.122 0 0.212" rpy="0 0 0"/>
+        <origin xyz="0.122 0 0.212" rpy="0 0 ${pi}"/>
     </joint>
     <link name="laser_frame">
@@ -26,5 +26,5 @@
         </collision>
         <xacro:inertial_cylinder mass="0.1" length="0.04" radius="0.05">
-            <origin xyz="0 0 0" rpy="0 0 3.1415"/>
+            <origin xyz="0 0 0" rpy="0 0 0"/>
         </xacro:inertial_cylinder>
     </link>

File: description/robot_core.xacro (robot description, xacro)
@@ -38,5 +38,5 @@
         <parent link="base_link"/>
         <child link="base_footprint"/>
-        <origin xyz="0 0 0" rpy="0 0 3.1415"/>
+        <origin xyz="0 0 0" rpy="0 0 0"/>
     </joint>
     <link name="base_footprint">
@@ -46,5 +46,5 @@
         <parent link="base_link"/>
         <child link="chassis"/>
-        <origin xyz="${-wheel_offset_x} 0 ${-wheel_offset_z}"/>
+        <origin xyz="${-wheel_offset_x} 0 ${-wheel_offset_z}" rpy="0 0 ${pi}" />
     </joint>
     <link name="chassis">

Commit message: wheel and lidar orientation fix

File: description/lidar.xacro (robot description, xacro)
@@ -1,8 +1,13 @@
 <?xml version="1.0"?>
 <robot xmlns:xacro="http://www.ros.org/wiki/xacro" >
+    <!-- <joint name="laser_joint" type="fixed">
+        <parent link="chassis"/>
+        <child link="laser_frame"/>
+        <origin xyz="0.122 0 0.212" rpy="0 0 ${pi}"/>
+    </joint> -->
     <joint name="laser_joint" type="fixed">
         <parent link="chassis"/>
         <child link="laser_frame"/>
-        <origin xyz="0.122 0 0.212" rpy="0 0 ${pi}"/>
+        <origin xyz="-0.122 0 0.212" rpy="0 0 0"/>
     </joint>
     <link name="laser_frame">

File: description/robot_core.xacro (robot description, xacro)
@@ -46,5 +46,5 @@
         <parent link="base_link"/>
         <child link="chassis"/>
-        <origin xyz="${-wheel_offset_x} 0 ${-wheel_offset_z}" rpy="0 0 ${pi}" />
+        <origin xyz="0 0 ${-wheel_offset_z}" rpy="0 0 ${pi}" />
     </joint>
     <link name="chassis">
@@ -73,5 +73,5 @@
         <parent link="base_link"/>
         <child link="left_wheel"/>
-        <origin xyz="0 ${wheel_offset_y} 0" rpy="-${pi/2} 0 0" />
+        <origin xyz="${-wheel_offset_x} ${wheel_offset_y} 0" rpy="-${pi/2} 0 0" />
         <axis xyz="0 0 1"/>
     </joint>
@@ -99,5 +99,5 @@
         <parent link="base_link"/>
         <child link="right_wheel"/>
-        <origin xyz="0 ${-wheel_offset_y} 0" rpy="${pi/2} 0 0" />
+        <origin xyz="${-wheel_offset_x} ${-wheel_offset_y} 0" rpy="${pi/2} 0 0" />
         <axis xyz="0 0 -1"/>
     </joint>
@@ -125,5 +125,5 @@
         <parent link="chassis"/>
         <child link="caster_wheel"/>
-        <origin xyz="${caster_wheel_offset_x} 0 ${caster_wheel_offset_z}"/>
+        <origin xyz="${-caster_wheel_offset_x} 0 ${caster_wheel_offset_z}"/>
     </joint>
     <link name="caster_wheel">

Commit message: lidar fix

File: description/lidar.xacro (robot description, xacro)
@@ -1,14 +1,14 @@
 <?xml version="1.0"?>
 <robot xmlns:xacro="http://www.ros.org/wiki/xacro" >
+    <joint name="laser_joint" type="fixed">
+        <parent link="chassis"/>
+        <child link="laser_frame"/>
+        <origin xyz="0.122 0 0.212" rpy="0 0 ${pi}"/>
+    </joint>
     <!-- <joint name="laser_joint" type="fixed">
         <parent link="chassis"/>
         <child link="laser_frame"/>
-        <origin xyz="0.122 0 0.212" rpy="0 0 ${pi}"/>
+        <origin xyz="-0.122 0 0.212" rpy="0 0 0"/>
     </joint> -->
-    <joint name="laser_joint" type="fixed">
-        <parent link="chassis"/>
-        <child link="laser_frame"/>
-        <origin xyz="-0.122 0 0.212" rpy="0 0 0"/>
-    </joint>
     <link name="laser_frame">
         <visual>

Commit message: reorientaition

File: description/lidar.xacro (robot description, xacro)
@@ -4,5 +4,5 @@
         <parent link="chassis"/>
         <child link="laser_frame"/>
-        <origin xyz="0.122 0 0.212" rpy="0 0 ${pi}"/>
+        <origin xyz="0.122 0 0.212" rpy="0 0 0"/>
     </joint>
     <!-- <joint name="laser_joint" type="fixed">

File: description/robot_core.xacro (robot description, xacro)
@@ -73,5 +73,5 @@
         <parent link="base_link"/>
         <child link="left_wheel"/>
-        <origin xyz="0 ${wheel_offset_y} 0" rpy="-${pi/2} 0 0" />
+        <origin xyz="${-wheel_offset_x} ${wheel_offset_y} 0" rpy="-${pi/2} 0 0" />
         <axis xyz="0 0 1"/>
     </joint>
@@ -99,5 +99,5 @@
         <parent link="base_link"/>
         <child link="right_wheel"/>
-        <origin xyz="0 ${-wheel_offset_y} 0" rpy="${pi/2} 0 0" />
+        <origin xyz="${-wheel_offset_x} ${-wheel_offset_y} 0" rpy="${pi/2} 0 0" />
         <axis xyz="0 0 -1"/>
     </joint>
@@ -125,5 +125,5 @@
         <parent link="chassis"/>
         <child link="caster_wheel"/>
-        <origin xyz="${caster_wheel_offset_x} 0 ${caster_wheel_offset_z}"/>
+        <origin xyz="${-caster_wheel_offset_x} 0 ${caster_wheel_offset_z}"/>
     </joint>
     <link name="caster_wheel">

Commit message: lidar fix

File: description/lidar.xacro (robot description, xacro)
@@ -4,5 +4,5 @@
         <parent link="chassis"/>
         <child link="laser_frame"/>
-        <origin xyz="0.122 0 0.212" rpy="0 0 0"/>
+        <origin xyz="0.122 0 0.212" rpy="0 0 ${pi}"/>
     </joint>
     <!-- <joint name="laser_joint" type="fixed">

Commit message: lidar fix

File: description/lidar.xacro (robot description, xacro)
@@ -4,11 +4,6 @@
         <parent link="chassis"/>
         <child link="laser_frame"/>
-        <origin xyz="0.122 0 0.212" rpy="0 0 ${pi}"/>
+        <origin xyz="-0.122 0 0.212" rpy="0 0 0"/>
     </joint>
-    <!-- <joint name="laser_joint" type="fixed">
-        <parent link="chassis"/>
-        <child link="laser_frame"/>
-        <origin xyz="-0.122 0 0.212" rpy="0 0 0"/>
-    </joint> -->
     <link name="laser_frame">
         <visual>

Commit message: orientatation fix

File: description/lidar.xacro (robot description, xacro)
@@ -4,6 +4,11 @@
         <parent link="chassis"/>
         <child link="laser_frame"/>
+        <origin xyz="0.122 0 0.212" rpy="0 0 ${pi}"/>
+    </joint>
+    <!-- <joint name="laser_joint" type="fixed">
+        <parent link="chassis"/>
+        <child link="laser_frame"/>
         <origin xyz="-0.122 0 0.212" rpy="0 0 0"/>
-    </joint>
+    </joint> -->
     <link name="laser_frame">
         <visual>

Commit message: rotate lidar

File: description/lidar.xacro (robot description, xacro)
@@ -1,8 +1,9 @@
 <?xml version="1.0"?>
 <robot xmlns:xacro="http://www.ros.org/wiki/xacro" >
+    <xacro:property name="pi" value="3.14159265359"/>
     <joint name="laser_joint" type="fixed">
         <parent link="chassis"/>
         <child link="laser_frame"/>
-        <origin xyz="0.122 0 0.212" rpy="0 0 0"/>
+        <origin xyz="0.122 0 0.212" rpy="0 0 ${pi}"/>
     </joint>
     <!-- <joint name="laser_joint" type="fixed">
@@ -37,5 +38,5 @@
         <material>Gazebo/Black</material>
         <sensor name="laser" type="ray">
-            <pose> 0 0 0 0 0 0 </pose>
+            <pose> 0 0 0 0 0 3.14159 </pose>
             <visualize>false</visualize>
             <update_rate>10</update_rate>

File: description/robot_core.xacro (robot description, xacro)
@@ -2,4 +2,5 @@
 <robot xmlns:xacro="http://www.ros.org/wiki/xacro" >
     <xacro:include filename="inertial_macros.xacro"/>
+    <xacro:property name="pi" value="3.14159265359"/>
     <xacro:property name="chassis_length" value="0.32"/>
     <xacro:property name="chassis_width" value="0.32"/>

Commit message: removed pi definition

File: description/lidar.xacro (robot description, xacro)
@@ -1,5 +1,5 @@
 <?xml version="1.0"?>
 <robot xmlns:xacro="http://www.ros.org/wiki/xacro" >
-    <xacro:property name="pi" value="3.14159265359"/>
+    <!-- <xacro:property name="pi" value="3.14159265359"/> -->
     <joint name="laser_joint" type="fixed">
         <parent link="chassis"/>

File: description/robot_core.xacro (robot description, xacro)
@@ -2,5 +2,5 @@
 <robot xmlns:xacro="http://www.ros.org/wiki/xacro" >
     <xacro:include filename="inertial_macros.xacro"/>
-    <xacro:property name="pi" value="3.14159265359"/>
+    <!-- <xacro:property name="pi" value="3.14159265359"/> -->
     <xacro:property name="chassis_length" value="0.32"/>
     <xacro:property name="chassis_width" value="0.32"/>

Commit message: rotated lidar 180 degrees

File: description/lidar.xacro (robot description, xacro)
@@ -5,5 +5,5 @@
         <parent link="chassis"/>
         <child link="laser_frame"/>
-        <origin xyz="0.122 0 0.212" rpy="0 0 ${pi}"/>
+        <origin xyz="0.122 0 0.212" rpy="0 0 0"/>
     </joint>
     <!-- <joint name="laser_joint" type="fixed">
